File: 5V Supply.sch (KiCad schematic (older format))
At the start: 4 parts, among them J1 Conn_01x11, U1 INA219AxD, U1 PoluluD24V10F5

Commit message: Add files via upload
Parts:
- U1: symbol Local:PoluluD24V10F5 -> 5V-Supply-rescue:PoluluD24V10F5-Local
Changed lines of the file:
@@
 $EndDescr
 $Comp
-L Local:PoluluD24V10F5 U1
+L 5V-Supply-rescue:PoluluD24V10F5-Local U1
 U 1 1 5DF4300F
 P 5350 2700
