File: PowerSupply2020.kicad_pcb (KiCad board)
At the start: 2 copper layers, 1 part, among them U1 LT1910ES8PBF

Commit message: Add files via upload
Parts:
- removed U1: LT1910ES8PBF, LT1910ES8PBF:SO-8_S
- added BZ1: Buzzer, Buzzer_Beeper:Buzzer_12x9.5RM7.6, F.Cu at (144.1, 67.9)
- added F1: 3544-2, Fuse:Fuse_Bourns_MF-RHT1000, F.Cu at (169.5, 62.2)
- added J1: DB9_Female, Connector_Dsub:DSUB-9_Female_Vertical_P2.77x2.84mm_MountingHoles, F.Cu at (39.4, 58.4)
- added J2: DB9_Female, Connector_Dsub:DSUB-9_Female_Vertical_P2.77x2.84mm_MountingHoles, F.Cu at (39.4, 92.1)
- added J3: DB9_Female, Connector_Dsub:DSUB-9_Female_Vertical_P2.77x2.84mm_MountingHoles, F.Cu at (39.4, 125.7)
- added J4: DB9_Female, Connector_Dsub:DSUB-9_Female_Vertical_P2.77x2.84mm_MountingHoles, F.Cu at (39.4, 159.4)
- added J5: Slave Address 1000000, Connector_Harwin:Harwin_Gecko-G125-FVX1205L0X_2x06_P1.25mm_Vertical, F.Cu at (161.3, 156.2)
- added J6: Slave Address 1000001, Connector_Harwin:Harwin_Gecko-G125-FVX1205L0X_2x06_P1.25mm_Vertical, F.Cu at (161.3, 139.9)
- added J7: Slave Address 1000010, Connector_Harwin:Harwin_Gecko-G125-FVX1205L0X_2x06_P1.25mm_Vertical, F.Cu at (161.3, 123.6)
- added J8: Slave Address 1000011, Connector_Harwin:Harwin_Gecko-G125-FVX1205L0X_2x06_P1.25mm_Vertical, F.Cu at (161.3, 107.3)
- added Q1: 2SC1815, Package_TO_SOT_THT:TO-92_Inline, F.Cu at (160.7, 66.7)
- added R1: 1 kΩ, Resistor_THT:R_Axial_DIN0204_L3.6mm_D1.6mm_P7.62mm_Horizontal, F.Cu at (151.8, 79.4)
- added R10: 10 kΩ, Resistor_THT:R_Axial_DIN0204_L3.6mm_D1.6mm_P7.62mm_Horizontal, F.Cu at (102.2, 55.2)
- added R11: 10 kΩ, Resistor_THT:R_Axial_DIN0204_L3.6mm_D1.6mm_P7.62mm_Horizontal, F.Cu at (141.6, 101.0)
- added R12: 10 kΩ, Resistor_THT:R_Axial_DIN0204_L3.6mm_D1.6mm_P7.62mm_Horizontal, F.Cu at (141.6, 94.6)
- added R2: 10 kΩ, Resistor_THT:R_Axial_DIN0204_L3.6mm_D1.6mm_P7.62mm_Horizontal, F.Cu at (111.1, 98.4)
- added R3: 10 kΩ, Resistor_THT:R_Axial_DIN0204_L3.6mm_D1.6mm_P7.62mm_Horizontal, F.Cu at (125.1, 104.8)
- added R4: 10 kΩ, Resistor_THT:R_Axial_DIN0204_L3.6mm_D1.6mm_P7.62mm_Horizontal, F.Cu at (111.1, 104.8)
- added R5: 10 kΩ, Resistor_THT:R_Axial_DIN0204_L3.6mm_D1.6mm_P7.62mm_Horizontal, F.Cu at (125.1, 98.4)
- added R6: 1 kΩ, Resistor_THT:R_Axial_DIN0204_L3.6mm_D1.6mm_P7.62mm_Horizontal, F.Cu at (144.1, 56.5)
- added REF**: R_Array_SIP4, Resistor_THT:R_Array_SIP4, F.Cu at (168.9, 87.6)
- added REF**: ProtoBoard, LocalFootprint:ProtoBoard, F.Cu at (80.6, 145.3)
- added REF**: ProtoBoard, LocalFootprint:ProtoBoard, F.Cu at (80.6, 111.7)
- added REF**: ProtoBoard, LocalFootprint:ProtoBoard, F.Cu at (80.6, 78.0)
- added REF**: ProtoBoard, LocalFootprint:ProtoBoard, F.Cu at (80.6, 44.4)
- added S1: TH_Sensor, Sensor:Aosong_DHT11_5.5x12.0_P2.54mm, F.Cu at (140.3, 48.9)
- added U2: L7805, Package_TO_SOT_THT:TO-92_Inline_Wide, F.Cu at (150.5, 87.0)
- added U3: Adafruit_Feather_M0_DOA, LocalFootprint:Adafruit_M0_DOA, F.Cu at (121.3, 67.9)
Routing:
- net Earth: track 0.00 -> 589.3 mm, vias 0 -> 4
- net /VOUT3: track 0.00 -> 301.7 mm, vias 0 -> 5
- net /VOUT4: track 0.00 -> 278.2 mm, vias 0 -> 1
- net (no net): track 0.00 -> 267.0 mm
- net /G_SW: track 0.00 -> 225.2 mm, vias 0 -> 5
- net /VOUT2: track 0.00 -> 204.8 mm, vias 0 -> 5
- net /VOUT1: track 0.00 -> 200.7 mm, vias 0 -> 3
- net /SDA: track 0.00 -> 167.0 mm, vias 0 -> 4
- net +5V: track 0.00 -> 158.5 mm, vias 0 -> 3
- net /RX: track 0.00 -> 155.7 mm, vias 0 -> 3
- net /TX: track 0.00 -> 154.6 mm, vias 0 -> 3
- net /PG_2: track 0.00 -> 152.3 mm, vias 0 -> 1
- net +12C: track 0.00 -> 151.3 mm, vias 0 -> 4
- net /SCL: track 0.00 -> 148.9 mm, vias 0 -> 2
- net /PG_1: track 0.00 -> 131.4 mm, vias 0 -> 1
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Other:
- board text added: "GND RX TX G_SW V1 V2 V3 V4"
