File: PowerSupply2020.sch (KiCad schematic (older format))
At the start: 5 parts, among them U1 LT1910ES8PBF

Commit message: Add files via upload
Parts:
- added C1: 10uF 50V, symbol Device:CP1
- added C2: 0.1 uF, symbol Device:CP1
- R1, R2: renamed from R?; symbol Device:R -> PowerSupply2020-rescue:R-Device
- R3: renamed from R?; value R -> 5.1 kΩ; symbol Device:R -> PowerSupply2020-rescue:R-Device
- R4: renamed from R?; value R -> 0.01 Ω; symbol Device:R -> PowerSupply2020-rescue:R-Device
Connections:
- net labels added: GND-power
- wire segments 2 -> 12
Changed lines of the file:
@@
 $EndDescr
+$Comp
+L PowerSupply2020-rescue:R-Device R1
+U 1 1 5DD62A55
+P 3200 1500
+F 0 "R1" H 3270 1546 50  0000 L CNN
+F 1 "R" H 3270 1455 50  0000 L CNN
+F 2 "" V 3130 1500 50  0001 C CNN
+F 3 "~" H 3200 1500 50  0001 C CNN
+	1    3200 1500
+	1    0    0    -1
+$EndComp
+$Comp
+L PowerSupply2020-rescue:R-Device R2
+U 1 1 5DD63099
+P 3150 1900
+F 0 "R2" H 3220 1946 50  0000 L CNN
+F 1 "R" H 3220 1855 50  0000 L CNN
+F 2 "" V 3080 1900 50  0001 C CNN
+F 3 "~" H 3150 1900 50  0001 C CNN
+	1    3150 1900
+	1    0    0    -1
+$EndComp
+$Comp
+L PowerSupply2020-rescue:R-Device R3
+U 1 1 5DD6340F
+P 3900 2300
+F 0 "R3" H 3970 2346 50  0000 L CNN
+F 1 "5.1 kΩ" H 3970 2255 50  0000 L CNN
+F 2 "" V 3830 2300 50  0001 C CNN
+F 3 "~" H 3900 2300 50  0001 C CNN
+	1    3900 2300
+	1    0    0    -1
+$EndComp
+$Comp
+L PowerSupply2020-rescue:R-Device R4
+U 1 1 5DD621EB
+P 7550 2000
+F 0 "R4" H 7620 2046 50  0000 L CNN
+F 1 "0.01 Ω" H 7620 1955 50  0000 L CNN
+F 2 "" V 7480 2000 50  0001 C CNN
+F 3 "~" H 7550 2000 50  0001 C CNN
+	1    7550 2000
+	1    0    0    -1
+$EndComp
+$Comp
+L PowerSupply2020-rescue:GND-power #PWR0102
+U 1 1 5DD66292
+P 4400 1950
+F 0 "#PWR0102" H 4400 1700 50  0001 C CNN
+F 1 "GND" V 4405 1822 50  0000 R CNN
+F 2 "" H 4400 1950 50  0001 C CNN
+F 3 "" H 4400 1950 50  0001 C CNN
+	1    4400 1950
+	0    1    1    0
+$EndComp
+Wire Wire Line
+	7000 1950 7100 1950
+Wire Wire Line
+	7100 1950 7100 1850
+Wire Wire Line
+	7100 1850 7550 1850
+Connection ~ 7100 1950
+$Comp
+L Device:CP1 C1
+U 1 1 5DF08086
+P 7100 2800
+F 0 "C1" H 7215 2846 50  0000 L CNN
+F 1 "10uF 50V" H 7215 2755 50  0000 L CNN
+F 2 "" H 7100 2800 50  0001 C CNN
+F 3 "~" H 7100 2800 50  0001 C CNN
+	1    7100 2800
+	1    0    0    -1
+$EndComp
+$Comp
+L PowerSupply2020-rescue:GND-power #PWR?
+U 1 1 5DF0B107
+P 7900 3250
+F 0 "#PWR?" H 7900 3000 50  0001 C CNN
+F 1 "GND-power" H 7905 3077 50  0000 C CNN
+F 2 "" H 7900 3250 50  0001 C CNN
+F 3 "" H 7900 3250 50  0001 C CNN
+	1    7900 3250
+	1    0    0    -1
+$EndComp
+Wire Wire Line
+	7900 3250 7100 3250
+Wire Wire Line
+	7100 3250 7100 2950
+Wire Wire Line
+	7100 1950 7100 2650
+$Comp
+L PowerSupply2020-rescue:+5V-power #PWR0101
+U 1 1 5DD65746
+P 3900 2550
+F 0 "#PWR0101" H 3900 2400 50  0001 C CNN
+F 1 "+5V" H 3915 2723 50  0000 C CNN
+F 2 "" H 3900 2550 50  0001 C CNN
+F 3 "" H 3900 2550 50  0001 C CNN
+	1    3900 2550
+	-1   0    0    1
+$EndComp
 $Comp
 L LT1910ES8PBF:LT1910ES8PBF U1
@@
 	1    0    0    -1
 $EndComp
+Wire Wire Line
+	3900 2450 3900 2550
 $Comp
-L Device:R R?
-U 1 1 5DD62A55
-P 3200 1500
-F 0 "R?" H 3270 1546 50  0000 L CNN
-F 1 "R" H 3270 1455 50  0000 L CNN
-F 2 "" V 3130 1500 50  0001 C CNN
-F 3 "~" H 3200 1500 50  0001 C CNN
-	1    3200 1500
+L Device:CP1 C2
+U 1 1 5DF10A46
+P 3450 2300
+F 0 "C2" H 3565 2346 50  0000 L CNN
+F 1 "0.1 uF" H 3565 2255 50  0000 L CNN
+F 2 "" H 3450 2300 50  0001 C CNN
+F 3 "~" H 3450 2300 50  0001 C CNN
+	1    3450 2300
 	1    0    0    -1
 $EndComp
 $Comp
-L Device:R R?
-U 1 1 5DD63099
-P 3550 1950
-F 0 "R?" H 3620 1996 50  0000 L CNN
-F 1 "R" H 3620 1905 50  0000 L CNN
-F 2 "" V 3480 1950 50  0001 C CNN
-F 3 "~" H 3550 1950 50  0001 C CNN
-	1    3550 1950
+L PowerSupply2020-rescue:GND-power #PWR?
+U 1 1 5DF12A55
+P 3450 2550
+F 0 "#PWR?" H 3450 2300 50  0001 C CNN
+F 1 "GND-power" H 3455 2377 50  0000 C CNN
+F 2 "" H 3450 2550 50  0001 C CNN
+F 3 "" H 3450 2550 50  0001 C CNN
+	1    3450 2550
 	1    0    0    -1
 $EndComp
-$Comp
-L Device:R R?
-U 1 1 5DD6340F
-P 3850 2650
-F 0 "R?" H 3920 2696 50  0000 L CNN
-F 1 "R" H 3920 2605 50  0000 L CNN
-F 2 "" V 3780 2650 50  0001 C CNN
-F 3 "~" H 3850 2650 50  0001 C CNN
-	1    3850 2650
-	1    0    0    -1
-$EndComp
-$Comp
-L Device:R R?
-U 1 1 5DD621EB
-P 4200 2300
-F 0 "R?" H 4270 2346 50  0000 L CNN
-F 1 "R" H 4270 2255 50  0000 L CNN
-F 2 "" V 4130 2300 50  0001 C CNN
-F 3 "~" H 4200 2300 50  0001 C CNN
-	1    4200 2300
-	1    0    0    -1
-$EndComp
-$Comp
-L power:+5V #PWR?
-U 1 1 5DD65746
-P 4200 2450
-F 0 "#PWR?" H 4200 2300 50  0001 C CNN
-F 1 "+5V" H 4215 2623 50  0000 C CNN
-F 2 "" H 4200 2450 50  0001 C CNN
-F 3 "" H 4200 2450 50  0001 C CNN
-	1    4200 2450
-	-1   0    0    1
-$EndComp
-$Comp
-L power:GND #PWR?
-U 1 1 5DD66292
-P 4400 1950
-F 0 "#PWR?" H 4400 1700 50  0001 C CNN
-F 1 "GND" V 4405 1822 50  0000 R CNN
-F 2 "" H 4400 1950 50  0001 C CNN
-F 3 "" H 4400 1950 50  0001 C CNN
-	1    4400 1950
-	0    1    1    0
-$EndComp
 Wire Wire Line
-	3900 2050 4400 2050
+	3450 2450 3450 2550
 Wire Wire Line
-	4400 2150 4200 2150
+	3900 2150 4400 2150
+Wire Wire Line
+	3450 2050 3450 2150
+Wire Wire Line
+	3450 2050 4400 2050
+Wire Wire Line
+	7000 2150 7550 2150
 $EndSCHEMATC

Commit message: Add files via upload
Parts:
- removed C1: 10uF 50V, symbol Device:CP1
- removed C2: 0.1 uF, symbol Device:CP1
- R?: renamed from R4; value 0.01 Ω -> R; symbol PowerSupply2020-rescue:R-Device -> Device:R
- R?: renamed from R1; symbol PowerSupply2020-rescue:R-Device -> Device:R
- R?: renamed from R2; symbol PowerSupply2020-rescue:R-Device -> Device:R
- R?: renamed from R3; value 5.1 kΩ -> R; symbol PowerSupply2020-rescue:R-Device -> Device:R
Connections:
- net labels removed: GND-power
- wire segments 12 -> 2
Changed lines of the file:
@@
 $EndDescr
-$Comp
-L PowerSupply2020-rescue:R-Device R1
-U 1 1 5DD62A55
-P 3200 1500
-F 0 "R1" H 3270 1546 50  0000 L CNN
-F 1 "R" H 3270 1455 50  0000 L CNN
-F 2 "" V 3130 1500 50  0001 C CNN
-F 3 "~" H 3200 1500 50  0001 C CNN
-	1    3200 1500
-	1    0    0    -1
-$EndComp
-$Comp
-L PowerSupply2020-rescue:R-Device R2
-U 1 1 5DD63099
-P 3150 1900
-F 0 "R2" H 3220 1946 50  0000 L CNN
-F 1 "R" H 3220 1855 50  0000 L CNN
-F 2 "" V 3080 1900 50  0001 C CNN
-F 3 "~" H 3150 1900 50  0001 C CNN
-	1    3150 1900
-	1    0    0    -1
-$EndComp
-$Comp
-L PowerSupply2020-rescue:R-Device R3
-U 1 1 5DD6340F
-P 3900 2300
-F 0 "R3" H 3970 2346 50  0000 L CNN
-F 1 "5.1 kΩ" H 3970 2255 50  0000 L CNN
-F 2 "" V 3830 2300 50  0001 C CNN
-F 3 "~" H 3900 2300 50  0001 C CNN
-	1    3900 2300
-	1    0    0    -1
-$EndComp
-$Comp
-L PowerSupply2020-rescue:R-Device R4
-U 1 1 5DD621EB
-P 7550 2000
-F 0 "R4" H 7620 2046 50  0000 L CNN
-F 1 "0.01 Ω" H 7620 1955 50  0000 L CNN
-F 2 "" V 7480 2000 50  0001 C CNN
-F 3 "~" H 7550 2000 50  0001 C CNN
-	1    7550 2000
-	1    0    0    -1
-$EndComp
-$Comp
-L PowerSupply2020-rescue:GND-power #PWR0102
-U 1 1 5DD66292
-P 4400 1950
-F 0 "#PWR0102" H 4400 1700 50  0001 C CNN
-F 1 "GND" V 4405 1822 50  0000 R CNN
-F 2 "" H 4400 1950 50  0001 C CNN
-F 3 "" H 4400 1950 50  0001 C CNN
-	1    4400 1950
-	0    1    1    0
-$EndComp
-Wire Wire Line
-	7000 1950 7100 1950
-Wire Wire Line
-	7100 1950 7100 1850
-Wire Wire Line
-	7100 1850 7550 1850
-Connection ~ 7100 1950
-$Comp
-L Device:CP1 C1
-U 1 1 5DF08086
-P 7100 2800
-F 0 "C1" H 7215 2846 50  0000 L CNN
-F 1 "10uF 50V" H 7215 2755 50  0000 L CNN
-F 2 "" H 7100 2800 50  0001 C CNN
-F 3 "~" H 7100 2800 50  0001 C CNN
-	1    7100 2800
-	1    0    0    -1
-$EndComp
-$Comp
-L PowerSupply2020-rescue:GND-power #PWR?
-U 1 1 5DF0B107
-P 7900 3250
-F 0 "#PWR?" H 7900 3000 50  0001 C CNN
-F 1 "GND-power" H 7905 3077 50  0000 C CNN
-F 2 "" H 7900 3250 50  0001 C CNN
-F 3 "" H 7900 3250 50  0001 C CNN
-	1    7900 3250
-	1    0    0    -1
-$EndComp
-Wire Wire Line
-	7900 3250 7100 3250
-Wire Wire Line
-	7100 3250 7100 2950
-Wire Wire Line
-	7100 1950 7100 2650
-$Comp
-L PowerSupply2020-rescue:+5V-power #PWR0101
-U 1 1 5DD65746
-P 3900 2550
-F 0 "#PWR0101" H 3900 2400 50  0001 C CNN
-F 1 "+5V" H 3915 2723 50  0000 C CNN
-F 2 "" H 3900 2550 50  0001 C CNN
-F 3 "" H 3900 2550 50  0001 C CNN
-	1    3900 2550
-	-1   0    0    1
-$EndComp
 $Comp
 L LT1910ES8PBF:LT1910ES8PBF U1
@@
 	1    0    0    -1
 $EndComp
-Wire Wire Line
-	3900 2450 3900 2550
 $Comp
-L Device:CP1 C2
-U 1 1 5DF10A46
-P 3450 2300
-F 0 "C2" H 3565 2346 50  0000 L CNN
-F 1 "0.1 uF" H 3565 2255 50  0000 L CNN
-F 2 "" H 3450 2300 50  0001 C CNN
-F 3 "~" H 3450 2300 50  0001 C CNN
-	1    3450 2300
+L Device:R R?
+U 1 1 5DD62A55
+P 3200 1500
+F 0 "R?" H 3270 1546 50  0000 L CNN
+F 1 "R" H 3270 1455 50  0000 L CNN
+F 2 "" V 3130 1500 50  0001 C CNN
+F 3 "~" H 3200 1500 50  0001 C CNN
+	1    3200 1500
 	1    0    0    -1
 $EndComp
 $Comp
-L PowerSupply2020-rescue:GND-power #PWR?
-U 1 1 5DF12A55
-P 3450 2550
-F 0 "#PWR?" H 3450 2300 50  0001 C CNN
-F 1 "GND-power" H 3455 2377 50  0000 C CNN
-F 2 "" H 3450 2550 50  0001 C CNN
-F 3 "" H 3450 2550 50  0001 C CNN
-	1    3450 2550
+L Device:R R?
+U 1 1 5DD63099
+P 3550 1950
+F 0 "R?" H 3620 1996 50  0000 L CNN
+F 1 "R" H 3620 1905 50  0000 L CNN
+F 2 "" V 3480 1950 50  0001 C CNN
+F 3 "~" H 3550 1950 50  0001 C CNN
+	1    3550 1950
 	1    0    0    -1
 $EndComp
+$Comp
+L Device:R R?
+U 1 1 5DD6340F
+P 3850 2650
+F 0 "R?" H 3920 2696 50  0000 L CNN
+F 1 "R" H 3920 2605 50  0000 L CNN
+F 2 "" V 3780 2650 50  0001 C CNN
+F 3 "~" H 3850 2650 50  0001 C CNN
+	1    3850 2650
+	1    0    0    -1
+$EndComp
+$Comp
+L Device:R R?
+U 1 1 5DD621EB
+P 4200 2300
+F 0 "R?" H 4270 2346 50  0000 L CNN
+F 1 "R" H 4270 2255 50  0000 L CNN
+F 2 "" V 4130 2300 50  0001 C CNN
+F 3 "~" H 4200 2300 50  0001 C CNN
+	1    4200 2300
+	1    0    0    -1
+$EndComp
+$Comp
+L power:+5V #PWR?
+U 1 1 5DD65746
+P 4200 2450
+F 0 "#PWR?" H 4200 2300 50  0001 C CNN
+F 1 "+5V" H 4215 2623 50  0000 C CNN
+F 2 "" H 4200 2450 50  0001 C CNN
+F 3 "" H 4200 2450 50  0001 C CNN
+	1    4200 2450
+	-1   0    0    1
+$EndComp
+$Comp
+L power:GND #PWR?
+U 1 1 5DD66292
+P 4400 1950
+F 0 "#PWR?" H 4400 1700 50  0001 C CNN
+F 1 "GND" V 4405 1822 50  0000 R CNN
+F 2 "" H 4400 1950 50  0001 C CNN
+F 3 "" H 4400 1950 50  0001 C CNN
+	1    4400 1950
+	0    1    1    0
+$EndComp
 Wire Wire Line
-	3450 2450 3450 2550
+	3900 2050 4400 2050
 Wire Wire Line
-	3900 2150 4400 2150
-Wire Wire Line
-	3450 2050 3450 2150
-Wire Wire Line
-	3450 2050 4400 2050
-Wire Wire Line
-	7000 2150 7550 2150
+	4400 2150 4200 2150
 $EndSCHEMATC

Commit message: Add files via upload
Parts:
- removed R? (x4): R, symbol Device:R
- removed U1: LT1910ES8PBF, LT1910ES8PBF:SO-8_S, symbol LT1910ES8PBF:LT1910ES8PBF
- added BZ1: Buzzer, symbol Device:Buzzer
- added D1, D2: 1N4448, Diode_THT:D_DO-35_SOD27_P7.62mm_Horizontal, symbol Diode:1N4448
- added F1: 3544-2, symbol Device:Fuse
- added H1: T-3 Min Activation, symbol Local:Activation
- added H2: G-switch Activation, symbol Local:Activation
- added H3: Conn_01x04_Male, symbol Connector:Conn_01x04_Male
- added J1: Slave Address 1000000, symbol Connector_Generic:Conn_01x11
- added J2: Slave Address 1000001, symbol Connector_Generic:Conn_01x11
- added J3: Slave Address 1000010, symbol Connector_Generic:Conn_01x11
- added J4: Slave Address 1000011, symbol Connector_Generic:Conn_01x11
- added J5, J6: DB9_Female, symbol Connector:DB9_Female
- added Q1: RS1E200BNTB, symbol Local:RS1E200BNTB
- added Q?: 2SC1815, Package_TO_SOT_THT:TO-92_Inline, symbol Transistor_BJT:2SC1815
- added R1, R10, R11, R2, R5 (x2), R6, R7, R8, R9: 10 kΩ, symbol Device:R_US
- added R3, R4: 1 kΩ, symbol Device:R_US
- added S1: TH_Sensor, symbol Local:AM2320
- added U1: Adafruit_Feather_M0_DOA, symbol Local:Adafruit_Feather_M0_DOA
- added U2: NL27WZ08USG, symbol Local:NL27WZ08USG
- added U3: L7805, symbol Regulator_Linear:L7805
- added U4, U5: Power, symbol Local:Power
Connections:
- net labels added: +12C, +12V, +3V3, BUZZ, EN_1, EN_2, EN_3, EN_4, EN_4_PRE, EN_5, EN_5_PRE, EN_6, EN_7, Earth, G_SW, PG_1, PG_2, PG_3, SCL, SDA, SP_FAN, SP_HEATER, VOUT1, VOUT2, VOUT3, VS
- net labels removed: GND
- wire segments 2 -> 187
Other:
- note added: "12/13/19"
- note added: "Camera Ejection Project"
- note added: "Soldering Project"
- note added: "Stevens RS Power Management Board 2019\n"

Commit message: Add files via upload
Parts:
- removed D1, D2: 1N4448, Diode_THT:D_DO-35_SOD27_P7.62mm_Horizontal, symbol Diode:1N4448
- removed H3: Conn_01x04_Male, symbol Connector:Conn_01x04_Male
- removed R10, R8, R9: 10 kΩ, symbol Device:R_US
- removed U2: NL27WZ08USG, symbol Local:NL27WZ08USG
- removed U4: Power, symbol Local:Power
- added J3, J4: DB9_Female, Connector_Dsub:DSUB-9_Female_Vertical_P2.77x2.84mm_MountingHoles, symbol Connector:DB9_Female
- BZ1: footprint (none) -> Buzzer_Beeper:Buzzer_12x9.5RM7.6
- F1: footprint (none) -> Fuse:Fuse_Bourns_MF-RHT1000
- H1, H2: symbol Local:Activation -> PowerSupply2020-rescue:Activation-Local
- J1: renamed from J5; footprint (none) -> Connector_Dsub:DSUB-9_Female_Vertical_P2.77x2.84mm_MountingHoles
- J2: renamed from J6; footprint (none) -> Connector_Dsub:DSUB-9_Female_Vertical_P2.77x2.84mm_MountingHoles
- J5: renamed from J1; footprint (none) -> Connector_Harwin:Harwin_Gecko-G125-FVX1205L0X_2x06_P1.25mm_Vertical
- J6: renamed from J2; footprint (none) -> Connector_Harwin:Harwin_Gecko-G125-FVX1205L0X_2x06_P1.25mm_Vertical
- J7: renamed from J3; footprint (none) -> Connector_Harwin:Harwin_Gecko-G125-FVX1205L0X_2x06_P1.25mm_Vertical
- J8: renamed from J4; footprint (none) -> Connector_Harwin:Harwin_Gecko-G125-FVX1205L0X_2x06_P1.25mm_Vertical
- Q2: renamed from Q1; symbol Local:RS1E200BNTB -> PowerSupply2020-rescue:RS1E200BNTB-Local
- R1: renamed from R3; footprint (none) -> Resistor_THT:R_Axial_DIN0204_L3.6mm_D1.6mm_P7.62mm_Horizontal
- R10: renamed from R11; footprint (none) -> Resistor_THT:R_Axial_DIN0204_L3.6mm_D1.6mm_P7.62mm_Horizontal
- R11: renamed from R1; footprint (none) -> Resistor_THT:R_Axial_DIN0204_L3.6mm_D1.6mm_P7.62mm_Horizontal
- R12: renamed from R2; footprint (none) -> Resistor_THT:R_Axial_DIN0204_L3.6mm_D1.6mm_P7.62mm_Horizontal
- R2, R3: renamed from R5; footprint (none) -> Resistor_THT:R_Axial_DIN0204_L3.6mm_D1.6mm_P7.62mm_Horizontal
- R4: renamed from R6; footprint (none) -> Resistor_THT:R_Axial_DIN0204_L3.6mm_D1.6mm_P7.62mm_Horizontal
- R5: renamed from R7; footprint (none) -> Resistor_THT:R_Axial_DIN0204_L3.6mm_D1.6mm_P7.62mm_Horizontal
- R6: renamed from R4; footprint (none) -> Resistor_THT:R_Axial_DIN0204_L3.6mm_D1.6mm_P7.62mm_Horizontal
- S1: footprint (none) -> Sensor:Aosong_DHT11_5.5x12.0_P2.54mm; symbol Local:AM2320 -> PowerSupply2020-rescue:AM2320-Local
- U1: renamed from U5; symbol Local:Power -> PowerSupply2020-rescue:Power-Local
- U2: renamed from U3; footprint (none) -> Package_TO_SOT_THT:TO-92_Inline_Wide
- U3: renamed from U1; footprint (none) -> LocalFootprint:Adafruit_M0_DOA; symbol Local:Adafruit_Feather_M0_DOA -> PowerSupply2020-rescue:Adafruit_Feather_M0_DOA-Local
- gave numbers to parts that had none: 1
Connections:
- net labels added: PG_4, RX, TX, VOUT4
- net labels removed: EN_4_PRE, EN_5, EN_5_PRE, EN_6, EN_7, SP_FAN, SP_HEATER
- wire segments 187 -> 144
Other:
- note added: "Project A"
- note added: "Project B"
- note added: "Project C"
- note added: "Project D"
- note added: "Stevens RS Power Management Board 2020\n"
- note removed: "Camera Ejection Project"
- note removed: "Soldering Project"
- note removed: "Stevens RS Power Management Board 2019\n"
- moved on the sheet: BZ1, F1, J1, J2, Q1, R1, R2, R3, R4, R5, R6, U2
